File: hardware/twisted/Twisted.kicad_pcb (KiCad board)
At the start: 4 copper layers, 14 x 32.7 mm, 50 parts, among them J1 battery connector, SW1 TS-1088-AR02016, SW2 TS-1088-AR02016, SW3 TS-1088-AR02016, SW4 TS-1088-AR02016, SW5 TS-1088-AR02016, SW6 TS-1088-AR02016, SW7 TS-1088-AR02016, U1 FXL6408UMX, U2 LW5233N11E, U3 BQ25628RYKR, U4 KH-1.27FH-2X10P-H4.3-SMT, U6 ESP32-S3FH4R2, U8 H5VU25UC, X1 SX16Y040000B71T001

Commit message: chore: cleanup schematics and PCBs polishing (no logic changes)
Parts:
- removed the R5 at (135.7, 87.6)
- added R4: 0402WGF1001TCE, lcsc:R0402, F.Cu at (135.6, 87.4)
- added TP10: GND, lcsc:2xTinyTestPoint, B.Cu at (143.0, 83.6)
- added TP7: USB_D+, lcsc:2xTinyTestPoint, B.Cu at (140.9, 85.1)
- added TP8: USB_D-, lcsc:2xTinyTestPoint, B.Cu at (142.0, 85.1)
- added TP9: VBUS, lcsc:2xTinyTestPoint, B.Cu at (139.9, 83.6)
- moved TP1 0.38 mm to (144.7, 90.4)
- moved R1 0.18 mm to (135.6, 82.2)
- renumbered C9 to C1, C12 to C10, C14 to C11, C17 to C12, C3 to C13, C4 to C14, C6 to C15, C20 to C16, C1 to C17, C16 to C18, C10 to C19, C11 to C2, C19 to C3, C7 to C4, C18 to C5, C13 to C6, C5 to C7, C15 to C8, C8 to C9, L2 to L1, L1 to L2, LED3 to LED2, R3 to R5, TP4 to TP1, TP5 to TP2, TP6 to TP3, TP1 to TP4, TP3 to TP5, TP2 to TP6, U3 to U1, U8 to U2, U4 to U3, U2 to U4, U1 to U5
Connections:
- U1 pad 4: Net-(U3-ILIM) -> CHARGE_DEFAULT_CURRENT
- U2 pad 1: unconnected-(U8-Pad1) -> GND
- U2 pad 10: unconnected-(U8-Pad10) -> GND
- U2 pad 5: unconnected-(U8-Pad5) -> GND
- U2 pad 6: unconnected-(U8-Pad6) -> GND
Routing:
- net Net-(U3-ILIM): track 18.5 -> 0.00 mm, vias 2 -> 0
- net CHARGE_DEFAULT_CURRENT: track 0.00 -> 18.2 mm, vias 0 -> 2
- net GPIO41: track 43.3 -> 35.9 mm
- net GPIO42: track 40.2 -> 33.6 mm
- net USB_D+: track 25.6 -> 28.4 mm, vias 0 -> 1
- net USB_D-: track 27.2 -> 29.9 mm, vias 0 -> 1
- net VBUS: track 48.0 -> 46.4 mm
- net +3.3V: track 24.6 -> 26.2 mm
- net UART_RX: track 4.65 -> 5.98 mm
- net VSYS: track 38.2 -> 39.2 mm
- net PMID: track 8.00 -> 8.61 mm
- net GPIO38: track 0.27 -> 0.00 mm, vias 1 -> 0
- net GND: track 25.6 -> 25.8 mm, vias 54 -> 59
Other:
- board text added: "Sep 2026 - Rev. 2"
- board text added: "Triax-Labs"
