File: hardware/twisted/Twisted.kicad_sch (KiCad schematic)
At the start: 52 parts, among them J1 battery connector, SW1 TS-1088-AR02016, SW2 TS-1088-AR02016, SW3 TS-1088-AR02016, SW4 TS-1088-AR02016, SW5 TS-1088-AR02016, SW6 TS-1088-AR02016, SW7 TS-1088-AR02016, U1 FXL6408UMX, U2 LW5233N11E, U3 BQ25628RYKR, U4 KH-1.27FH-2X10P-H4.3-SMT, U6 ESP32-S3FH4R2, U8 H5VU25UC, X1 SX16Y040000B71T001

Commit message: chore: cleanup schematics and PCBs polishing (no logic changes)
Parts:
- removed LED2: KT-0603R, lcsc:LED-SMD_L1.6-W0.8-R-RD, symbol lcsc:KT-0603R
- removed R4: 0402WGF4701TCE, lcsc:R0402, symbol lcsc:0402WGF4701TCE
- removed R5: 0402WGF1001TCE, lcsc:R0402, symbol lcsc:0402WGF1001TCE
- added LED1: KT-0603R, lcsc:LED-SMD_L1.6-W0.8-R-RD, symbol lcsc:KT-0603R
- added R3: 0402WGF4701TCE, lcsc:R0402, symbol lcsc:0402WGF4701TCE
- added R4: 0402WGF1001TCE, lcsc:R0402, symbol lcsc:0402WGF1001TCE
- added TP10: GND, lcsc:2xTinyTestPoint, symbol Connector:TestPoint
- added TP7: USB_D+, lcsc:2xTinyTestPoint, symbol Connector:TestPoint
- added TP8: USB_D-, lcsc:2xTinyTestPoint, symbol Connector:TestPoint
- added TP9: VBUS, lcsc:2xTinyTestPoint, symbol Connector:TestPoint
- renumbered C9 to C1, C12 to C10, C14 to C11, C17 to C12, C3 to C13, C4 to C14, C6 to C15, C20 to C16, C1 to C17, C16 to C18, C10 to C19, C11 to C2, C19 to C3, C7 to C4, C18 to C5, C13 to C6, C5 to C7, C15 to C8, C8 to C9, L2 to L1, L1 to L2, LED3 to LED2, LED1 to LED3, R3 to R5, TP4 to TP1, TP5 to TP2, TP6 to TP3, TP1 to TP4, TP3 to TP5, TP2 to TP6, U3 to U1, U8 to U2, U4 to U3, U2 to U4, U1 to U5
Connections:
- net BAT_STAT: now also LED1.2 (K)
- net GND: now also U2.1, U2.10, U2.5, U2.6, R4.1, TP10.1
- net USB_D+: now also TP7.1
- net USB_D-: now also TP8.1
- net VBUS: now also R3.2, TP9.1
- net CHARGE_DEFAULT_CURRENT: now reaches U1.4 (ILIM)
- net CHARGE_DEFAULT_CURRENT: now also R4.2
- new net: LED1.1 (A), R3.1
- no-connect marks 29 -> 25
Other:
- note added: "7-bit Address: 0x43"
- note added: "7-bit Address: 0x6A"
- note added: "Battery Management"
- note added: "Expansion Header (Twisted Bus)"
- note added: "Pin Definition for Internal Devices"
- note added: "STAT indicates the charging status. The LED should be placed on the front. (IF USED)"
- note removed: "Expansion Header"
- note removed: "STAT indicates the charging status. The LED should be placed on the front."
- moved on the sheet: C19, C3, C4, C5, C6, C7, C9, J1, L1, LCD1, LED2, R1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
