File: hardware/twisted-listen/Twisted-Listen-Rev2.kicad_pcb (KiCad board)
At the start: 4 copper layers, 14 x 32.7 mm, 55 parts, among them CN1 SM02B-SRSS-TB, U1 LPA2103AQVF, U2 TCA9536DTMR, U3 LP5910-1.8DRVR, U4 ES8316, U5 KH-1.27FH-2X10P-H4.3-SMT

Commit message: chore: cleanup schematics and PCBs polishing (no logic changes)
Parts:
- added C9: CC0402KRX7R7BB104, lcsc:C0402, F.Cu at (147.0, 90.0)
- moved L1 1.70 mm to (142.2, 82.0), turned to 180 degrees
- moved C12 1.11 mm to (137.5, 93.5)
- moved C14 1.00 mm to (137.9, 94.9)
- moved C15 1.00 mm to (137.9, 95.9)
- moved R10 1.00 mm to (135.7, 94.9)
- moved R11 1.00 mm to (135.7, 95.9)
- moved C33 0.94 mm to (144.5, 82.1)
- moved C4 0.69 mm to (146.3, 82.1), turned to 0 degrees
- moved C13 0.55 mm to (139.6, 94.9)
- moved C6 0.47 mm to (135.7, 88.4)
- moved C16 0.41 mm to (146.0, 94.0)
- moved C3 0.39 mm to (135.7, 90.6), turned to 180 degrees
- moved TP3 0.25 mm to (136.1, 91.8)
- moved U3 0.19 mm to (145.5, 95.6)
- moved L2 0.16 mm to (138.7, 93.0)
Connections:
- net EXT_PIN10 renamed GPIO12
- net EXT_PIN12 renamed GPIO10
- net EXT_PIN5 renamed GPIO15
- net EXT_PIN7 renamed GPIO13
- net EXT_PIN8 renamed GPIO14
- C14 pad 2: EXT_PIN16 -> GPIO17
- C15 pad 2: EXT_PIN14 -> GPIO16
- H1 pad 10: EXT_PIN9 -> GPIO11
- H1 pad 12: EXT_PIN11 -> GPIO9
- H1 pad 13: EXT_PIN14 -> GPIO8
- H1 pad 14: EXT_PIN13 -> GPIO7
- H1 pad 15: EXT_PIN16 -> GPIO6
- H1 pad 16: EXT_PIN15 -> GPIO5
- H1 pad 17: EXT_PIN18 -> GPIO4
- H1 pad 18: EXT_PIN17 -> GPIO3
- H1 pad 19: EXT_PIN20 -> GPIO2
- H1 pad 20: EXT_PIN19 -> GPIO1
- H1 pad 3: EXT_PIN4 -> GPIO17
- H1 pad 5: EXT_PIN6 -> GPIO16
- R10 pad 1: EXT_PIN16 -> GPIO17
- R11 pad 1: EXT_PIN14 -> GPIO16
- R5 pad 1: EXT_PIN9 -> GPIO5
- R6 pad 1: EXT_PIN11 -> GPIO4
- R7 pad 1: EXT_PIN13 -> GPIO2
- R8 pad 1: EXT_PIN17 -> GPIO1
- R9 pad 1: EXT_PIN15 -> GPIO3
- U2 pad 5: EXT_PIN16 -> GPIO17
- U2 pad 6: EXT_PIN14 -> GPIO16
- U4 pad 1: EXT_PIN16 -> GPIO17
- U4 pad 32: EXT_PIN14 -> GPIO16
- U5 pad 11: EXT_PIN11 -> GPIO9
- U5 pad 13: EXT_PIN13 -> GPIO7
- U5 pad 14: EXT_PIN14 -> GPIO8
- U5 pad 15: EXT_PIN15 -> GPIO5
- U5 pad 16: EXT_PIN16 -> GPIO6
- U5 pad 17: EXT_PIN17 -> GPIO3
- U5 pad 18: EXT_PIN18 -> GPIO4
- U5 pad 19: EXT_PIN19 -> GPIO1
- U5 pad 20: EXT_PIN20 -> GPIO2
- U5 pad 4: EXT_PIN4 -> GPIO17
- U5 pad 6: EXT_PIN6 -> GPIO16
- U5 pad 9: EXT_PIN9 -> GPIO11
Routing:
- net GPIO17: track 0.00 -> 40.5 mm, vias 0 -> 5
- net EXT_PIN14: track 40.4 -> 0.00 mm, vias 4 -> 0
- net EXT_PIN16: track 40.4 -> 0.00 mm, vias 4 -> 0
- net GPIO16: track 0.00 -> 39.3 mm, vias 0 -> 5
- net GPIO2: track 0.00 -> 24.4 mm, vias 0 -> 3
- net GPIO4: track 0.00 -> 24.4 mm, vias 0 -> 3
- net GPIO5: track 0.00 -> 24.0 mm, vias 0 -> 3
- net GPIO3: track 0.00 -> 24.0 mm, vias 0 -> 3
- net +1V8: track 31.6 -> 10.8 mm
- net GPIO1: track 0.00 -> 19.1 mm, vias 0 -> 3
- net EXT_PIN9: track 19.0 -> 0.00 mm, vias 2 -> 0
- net EXT_PIN11: track 18.9 -> 0.00 mm, vias 2 -> 0
- net EXT_PIN15: track 18.9 -> 0.00 mm, vias 2 -> 0
- net EXT_PIN17: track 18.8 -> 0.00 mm, vias 2 -> 0
- net EXT_PIN13: track 18.8 -> 0.00 mm, vias 2 -> 0
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- added copper zone on In2.Cu, net +1V8
