File: hardware/twisted-listen/Twisted-Listen-Rev2.kicad_sch (KiCad schematic)
At the start: 55 parts, among them CN1 SM02B-SRSS-TB, U1 LPA2103AQVF, U2 TCA9536DTMR, U3 LP5910-1.8DRVR, U4 ES8316, U5 KH-1.27FH-2X10P-H4.3-SMT

Commit message: chore: cleanup schematics and PCBs polishing (no logic changes)
Parts:
- added C9: CC0402KRX7R7BB104, lcsc:C0402, symbol lcsc:CC0402KRX7R7BB104
- JP1: value SolderJumper_3_Bridged12 -> I2C Address Select
- TP1: value TestPoint -> 1.8V
- TP4: value TestPoint -> Extra GPIO
Connections:
- net EXT_PIN4 is gone; now on net GPIO17: H1.3, U5.4
- net EXT_PIN6 is gone; now on net GPIO16: H1.5, U5.6
- net +3.3V: now also C9.2
- net GND: now also C9.1
- net EXT_PIN10 renamed GPIO12
- net EXT_PIN11 renamed GPIO9
- net GPIO9: no longer R6.1
- net EXT_PIN12 renamed GPIO10
- net EXT_PIN13 renamed GPIO7
- net GPIO7: no longer R7.1
- net EXT_PIN14 renamed GPIO16
- net GPIO16: no longer H1.13, U5.14
- net EXT_PIN15 renamed GPIO5
- net GPIO5: now also R5.1; no longer R9.1
- net EXT_PIN16 renamed GPIO17
- net GPIO17: no longer H1.15, U5.16
- net EXT_PIN17 renamed GPIO3
- net GPIO3: now also R9.1; no longer R8.1
- net EXT_PIN18 renamed GPIO4
- net GPIO4: now also R6.1
- net EXT_PIN19 renamed GPIO1
- net GPIO1: now also R8.1
- net EXT_PIN20 renamed GPIO2
- net GPIO2: now also R7.1
- net EXT_PIN5 renamed GPIO15
- net EXT_PIN7 renamed GPIO13
- net EXT_PIN8 renamed GPIO14
- net EXT_PIN9 renamed GPIO11
- net GPIO11: no longer R5.1
- new net GPIO6: H1.15, U5.16
- new net GPIO8: H1.13, U5.14
Other:
- note added: "/ FREE (INT/CS)"
- note added: "1.8v Regulator"
- note added: "3.5mm Headphone Jack"
- note added: "Built-in Microphone (used to spy on you)"
- note added: "Decoupling"
- note added: "Extra Controls Over I2C"
- note added: "FREE (INT/CS)"
- note added: "I2C: SDA"
- note added: "I2S: ADC_DOUT"
- note added: "I2S: DAC_DIN"
- note added: "I2S: DLR_CLK"
- note added: "I2S: M_CLK"
- note added: "I2S: S_CLK"
- note added: "Loudspeaker Amplifier -> Shutdown using the GPIO expander"
- note added: "Pin Assignments"
- note added: "Pull-ups Needed I2C: SCL"
- note added: "SDIO: CS/ D3"
- note added: "SDIO: D1"
- note added: "SDIO: D2"
- note added: "SPI/SDIO: MISO / D0"
- note added: "SPI/SDIO: MOSI / CMD"
- note added: "SPI/SDIO: SCK"
- note added: "Twisted Header Bus"
- note added: "UART: RX"
- note added: "UART: TX"
- moved on the sheet: Audio1, C1, C10, C11, C12, C13, C16, C17, C18, C19, C2, C20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
